Commit message: - initial update for urdf with the new geometry

File: src/my_robot_description/urdf/cubic_doggo.ros2_control.xacro (robot description, xacro)
@@ -3,6 +3,6 @@
     <ros2_control name="cubic_doggo_controller" type="system">
         <hardware>
-            <!--plugin>mock_components/GenericSystem</plugin-->
-            <plugin>cubic_doggo_namespace/HardwareInterfaceU2D2_cubic_doggo</plugin>
+            <plugin>mock_components/GenericSystem</plugin>
+            <!--plugin>cubic_doggo_namespace/HardwareInterfaceU2D2_cubic_doggo</plugin-->
             <param name="servo1_channel_FL">11</param>
             <param name="servo2_channel_FL">12</param>

File: src/my_robot_description/urdf/cubic_doggo.urdf.xacro (robot description, xacro)
@@ -2,5 +2,6 @@
 <robot name="cubic_doggo" xmlns:xacro="http://www.ros.org/wiki/xacro">
     <xacro:include filename="common_properties.xacro"/>
-    <xacro:include filename="cubic_doggo_leg.xacro"/>
+    <xacro:include filename="cubic_doggo_legF.xacro"/>
+    <xacro:include filename="cubic_doggo_legB.xacro"/>
     <xacro:include filename="cubic_doggo.ros2_control.xacro"/>
 <!-- ================================================================================================================================== -->
@@ -9,5 +10,5 @@
         <visual>
             <geometry>
-                <mesh filename="package://my_robot_description/mesh/CADv0.1/basePlateTorsoUpper.stl" scale="0.001 0.001 0.001"/>
+                <mesh filename="package://my_robot_description/mesh/CADv1/baseTorso.stl" scale="0.001 0.001 0.001"/>
             </geometry>
             <origin xyz="0 0 0" rpy="0 0 0"/>
@@ -26,4 +27,25 @@
         <child  link="base_link"/>
         <origin xyz="0 0 0" rpy="0 0 0"/>
+    </joint>
+    <link name="base_plate_B">
+        <visual>
+            <geometry>
+                <mesh filename="package://my_robot_description/mesh/CADv1/basePlate.stl" scale="0.001 0.001 0.001"/>
+            </geometry>
+            <origin xyz="0 0 0" rpy="0 0 0"/>
+            <material name="grey"/>
+        </visual>
+        <collision>
+            <geometry>
+                <box size="0.141 0.036 0.004"/>
+            </geometry>
+            <origin xyz="0 0.018 0.002" rpy="0 0 0"/>
+        </collision>
+        <xacro:box_inertia m="0.0336" x="0.141" y="0.036" z="0.004" o_xyz="0 0.018 0.002" o_rpy="0 0 0"/>
+    </link>
+    <joint name="torso_base_plate_B" type="fixed">
+        <parent link="base_link"/>
+        <child  link="base_plate_B"/>
+        <origin xyz="0 -0.066 0.004" rpy="0 0 0"/>
     </joint>
     <link name="base_plate_F">
@@ -46,32 +68,11 @@
         <parent link="base_link"/>
         <child  link="base_plate_F"/>
-        <origin xyz="0 -0.066 0.004" rpy="0 0 0"/>
-    </joint>
-    <link name="base_plate_B">
-        <visual>
-            <geometry>
-                <mesh filename="package://my_robot_description/mesh/CADv1/basePlate.stl" scale="0.001 0.001 0.001"/>
-            </geometry>
-            <origin xyz="0 0 0" rpy="0 0 0"/>
-            <material name="grey"/>
-        </visual>
-        <collision>
-            <geometry>
-                <box size="0.141 0.036 0.004"/>
-            </geometry>
-            <origin xyz="0 0.018 0.002" rpy="0 0 0"/>
-        </collision>
-        <xacro:box_inertia m="0.0336" x="0.141" y="0.036" z="0.004" o_xyz="0 0.018 0.002" o_rpy="0 0 0"/>
-    </link>
-    <joint name="torso_base_plate_B" type="fixed">
-        <parent link="base_link"/>
-        <child  link="base_plate_B"/>
-        <origin xyz="0 0.09 0.004" rpy="0 0 0"/>
+        <origin xyz="0 0.091 0.004" rpy="0 0 ${urdf_pi}"/>
     </joint>
 <!-- ================================================================================================================================== -->
-    <xacro:doggo_leg prefix='FL'/>
-    <xacro:doggo_leg prefix='FR'/>
-    <xacro:doggo_leg prefix='BL'/>
-    <xacro:doggo_leg prefix='BR'/>
+    <xacro:doggo_legF prefix='FL'/>
+    <xacro:doggo_legF prefix='FR'/>
+    <xacro:doggo_legB prefix='BL'/>
+    <xacro:doggo_legB prefix='BR'/>
 <!-- ================================================================================================================================== -->
 </robot>

Commit message: - the robot can now move correctly again with the updated urdf

File: src/my_robot_description/urdf/cubic_doggo.ros2_control.xacro (robot description, xacro)
@@ -3,6 +3,6 @@
     <ros2_control name="cubic_doggo_controller" type="system">
         <hardware>
-            <plugin>mock_components/GenericSystem</plugin>
-            <!--plugin>cubic_doggo_namespace/HardwareInterfaceU2D2_cubic_doggo</plugin-->
+            <!--plugin>mock_components/GenericSystem</plugin-->
+            <plugin>cubic_doggo_namespace/HardwareInterfaceU2D2_cubic_doggo</plugin>
             <param name="servo1_channel_FL">11</param>
             <param name="servo2_channel_FL">12</param>

File: src/my_robot_description/urdf/cubic_doggo_legB.xacro (robot description, xacro)
@@ -129,5 +129,6 @@
             <origin xyz="0 ${-servo_y/2} 0" rpy="0 ${rflc*urdf_pi/2} 0"/>
         </collision>
-        <xacro:box_inertia m="0.0572" x="${servo_x}" y="${servo_y}" z="${servo_z}" o_xyz="0 ${-servo_y/2} 0" o_rpy="0 ${rflc*urdf_pi/2} 0"/>
+        <xacro:box_inertia m="0.0572" x="${servo_x}" y="${servo_y}" z="${servo_z}"
+                           o_xyz="0 ${-servo_y/2} 0" o_rpy="0 ${rflc*urdf_pi/2} 0"/>
     </link>
     <joint name="servo2_holder_servo2_${prefix}" type="fixed">
@@ -155,6 +156,6 @@
         <parent link="servo2_${prefix}"/>
         <child  link="servo2_padding_${prefix}"/>
-        <origin xyz="${rflc*(servo_z/2+0.002)} -0.01125 0" rpy="0 0 0"/>
-        <axis xyz="${rflc} 0 0"/>
+        <origin xyz="${rflc*(servo_z/2+0.002)} -0.01125 0" rpy="${-3*urdf_pi/8} 0 0"/>
+        <axis xyz="${-rflc} 0 0"/>
         <limit effort="1000.0" velocity="20.0" lower="${urdf_pi - 2*urdf_pi/6 - rflc*urdf_pi/6}"
                                                upper="${urdf_pi + 2*urdf_pi/6 - rflc*urdf_pi/6}"/>
@@ -168,5 +169,5 @@
             </geometry>
             <material name="blue"/>
-            <origin xyz="0 0 0" rpy="${-rflc*urdf_pi/2} 0 ${-urdf_pi/2}"/>
+            <origin xyz="0 0 0" rpy="${rflc*urdf_pi/2} 0 ${-urdf_pi/2}"/>
         </visual>
         <collision>
@@ -174,13 +175,13 @@
                 <box size="0.032 0.040 0.006"/>
             </geometry>
-            <origin xyz="${rflc*0.003} -0.016 0" rpy="${-rflc*urdf_pi/2} 0 ${-urdf_pi/2}"/>
+            <origin xyz="${-rflc*0.003} -0.016 0" rpy="${rflc*urdf_pi/2} 0 ${-urdf_pi/2}"/>
         </collision>
         <xacro:box_inertia m="0.0085" x="0.032" y="0.040" z="0.006"
-                           o_xyz="${rflc*0.003} -0.016 0" o_rpy="${-rflc*urdf_pi/2} 0 ${-urdf_pi/2}"/>
+                           o_xyz="${-rflc*0.003} -0.016 0" o_rpy="${rflc*urdf_pi/2} 0 ${-urdf_pi/2}"/>
     </link>
     <joint name="servo2_padding_inner_thigh_${prefix}" type="fixed">
         <parent link="servo2_padding_${prefix}"/>
         <child  link="inner_thigh_${prefix}"/>
-        <origin xyz="${rflc*0.004} 0.016 0" rpy="0 0 0"/>
+        <origin xyz="${rflc*0.004} 0 -0.016" rpy="${-3*urdf_pi/8} 0 ${urdf_pi}"/>
     </joint>
     <link name="outer_thigh_${prefix}">
@@ -190,5 +191,5 @@
             </geometry>
             <material name="blue"/>
-            <origin xyz="0 0 0" rpy="${-urdf_pi/2} ${urdf_pi/2-rflc*urdf_pi/2} ${-rflc*urdf_pi/2}"/>
+            <origin xyz="0 0 0" rpy="${-urdf_pi/2} ${urdf_pi/2+rflc*urdf_pi/2} ${rflc*urdf_pi/2}"/>
         </visual>
         <collision>
@@ -196,13 +197,13 @@
                 <box size="0.040 0.032 0.006"/>
             </geometry>
-            <origin xyz="${rflc*0.003} -0.0475 0" rpy="${-urdf_pi/2} ${urdf_pi/2-rflc*urdf_pi/2} ${-rflc*urdf_pi/2}"/>
+            <origin xyz="${-rflc*0.003} -0.0475 0" rpy="${-urdf_pi/2} ${urdf_pi/2+rflc*urdf_pi/2} ${rflc*urdf_pi/2}"/>
         </collision>
         <xacro:box_inertia m="0.0113" x="0.040" y="0.032" z="0.006"
-                           o_xyz="${rflc*0.003} -0.0475 0" o_rpy="${-urdf_pi/2} ${urdf_pi/2-rflc*urdf_pi/2} ${-rflc*urdf_pi/2}"/>
+                           o_xyz="${-rflc*0.003} -0.0475 0" o_rpy="${-urdf_pi/2} ${urdf_pi/2+rflc*urdf_pi/2} ${rflc*urdf_pi/2}"/>
     </link>
     <joint name="inner_thigh_outer_thigh_${prefix}" type="fixed">
         <parent link="inner_thigh_${prefix}"/>
         <child  link="outer_thigh_${prefix}"/>
-        <origin xyz="${rflc*0.028} 0 0" rpy="0 0 0"/>
+        <origin xyz="${-rflc*0.028} 0 0" rpy="0 0 0"/>
     </joint>
     <link name="servo3_${prefix}">
@@ -211,5 +212,5 @@
                 <box size="${servo_x} ${servo_y} ${servo_z}"/>
             </geometry>
-            <origin xyz="0 ${-servo_y/2} 0" rpy="0 ${rflc*urdf_pi/2} 0"/>
+            <origin xyz="0 ${-servo_y/2} 0" rpy="0 ${-rflc*urdf_pi/2} 0"/>
             <material name="black"/>
         </visual>
@@ -218,13 +219,13 @@
                 <box size="${servo_x} ${servo_y} ${servo_z}"/>
             </geometry>
-            <origin xyz="0 ${-servo_y/2} 0" rpy="0 ${rflc*urdf_pi/2} 0"/>
+            <origin xyz="0 ${-servo_y/2} 0" rpy="0 ${-rflc*urdf_pi/2} 0"/>
         </collision>
         <xacro:box_inertia m="${0.0572+0.0113+0.0078}" x="${servo_x}" y="${servo_y}" z="${servo_z}"
-                           o_xyz="0 ${-servo_y/2} 0" o_rpy="0 ${rflc*urdf_pi/2} 0"/>
+                           o_xyz="0 ${-servo_y/2} 0" o_rpy="0 ${-rflc*urdf_pi/2} 0"/>
     </link>
     <joint name="outer_thigh_servo3_${prefix}" type="fixed">
         <parent link="outer_thigh_${prefix}"/>
         <child  link="servo3_${prefix}"/>
-        <origin xyz="${rflc*(servo_y/2-0.006-0.0025)} -0.004 0" rpy="0 0 0"/>
+        <origin xyz="${-rflc*(servo_y/2-0.006-0.0025)} -0.004 0" rpy="0 0 0"/>
     </joint>
     <link name="calfFeet_${prefix}">
@@ -248,5 +249,5 @@
         <parent link="servo3_${prefix}"/>
         <child  link="calfFeet_${prefix}"/>
-        <origin xyz="${rflc*(-servo_z/2-0.002-0.0025)} ${-0.086+0.004} 0" rpy="0 0 0"/>
+        <origin xyz="${-rflc*(-servo_z/2-0.002-0.0025)} ${-0.086+0.004} 0" rpy="0 0 0"/>
         <axis xyz="${-rflc} 0 0"/>
         <limit effort="1000.0" velocity="20.0" lower="${5*urdf_pi/8}" upper="${11*urdf_pi/8}"/>
@@ -258,5 +259,5 @@
                 <mesh filename="package://my_robot_description/mesh/CADv1/calfJoint.stl" scale="0.001 0.001 0.001"/>
             </geometry>
-            <origin xyz="0 0 0" rpy="${urdf_pi/2} 0 ${-rflc*urdf_pi/2}"/>
+            <origin xyz="0 0 0" rpy="${urdf_pi/2} 0 ${rflc*urdf_pi/2}"/>
             <material name="white"/>
         </visual>
@@ -265,13 +266,13 @@
                 <box size="0.022 0.053 0.007"/>
             </geometry>
-            <origin xyz="${-rflc*0.0005} 0 0.0155" rpy="${urdf_pi/2} 0 ${-rflc*urdf_pi/2}"/>
+            <origin xyz="${rflc*0.0005} 0 0.0155" rpy="${urdf_pi/2} 0 ${rflc*urdf_pi/2}"/>
         </collision>
         <xacro:box_inertia m="${0.0047+0.0015}" x="0.022" y="0.053" z="0.007"
-                           o_xyz="${-rflc*0.0005} 0 0.0155" o_rpy="${urdf_pi/2} 0 ${-rflc*urdf_pi/2}"/>
+                           o_xyz="${rflc*0.0005} 0 0.0155" o_rpy="${urdf_pi/2} 0 ${rflc*urdf_pi/2}"/>
     </link>
     <joint name="servo3_calfJoint_${prefix}" type="revolute">
         <parent link="servo3_${prefix}"/>
         <child  link="calfJoint_${prefix}"/>
-        <origin xyz="${rflc*(-servo_z/2-0.002-0.0025)} ${-0.01-0.0025/2} 0" rpy="0 0 0"/>
+        <origin xyz="${-rflc*(-servo_z/2-0.002-0.0025)} ${-0.01-0.0025/2} 0" rpy="0 0 0"/>
         <axis xyz="${-rflc} 0 0"/>
         <mimic joint="servo3_calfFeet_${prefix}" multiplier="1.0" offset="0.0"/>
