Commit message: - debug IK solution not found, just stride/lift reversed - redon cubic_doggo_legB.xacro rigorously peice by peice

File: src/my_robot_description/urdf/cubic_doggo_legB.xacro (robot description, xacro)
@@ -6,23 +6,13 @@
     <xacro:property name="servo_y" value="0.0465"/>
     <xacro:property name="servo_z" value="0.034"/>
-    <xacro:if value="${prefix == 'FL'}">
-        <xacro:property name="rflc"              value=" 1"/>
-        <xacro:property name="base_plate"        value="base_plate_F"/>
-        <xacro:property name="servo1_holder_xyz" value="-0.052 0.018 0.004"/>
-    </xacro:if>
-    <xacro:if value="${prefix == 'FR'}">
+    <xacro:if value="${prefix == 'BL'}">
         <xacro:property name="rflc"              value="-1"/>
-        <xacro:property name="base_plate"        value="base_plate_F"/>
+        <xacro:property name="base_plate"        value='base_plate_B'/>
         <xacro:property name="servo1_holder_xyz" value=" 0.052 0.018 0.004"/>
     </xacro:if>
-    <xacro:if value="${prefix == 'BL'}">
+    <xacro:if value="${prefix == 'BR'}">
         <xacro:property name="rflc"              value=" 1"/>
         <xacro:property name="base_plate"        value='base_plate_B'/>
         <xacro:property name="servo1_holder_xyz" value="-0.052 0.018 0.004"/>
-    </xacro:if>
-    <xacro:if value="${prefix == 'BR'}">
-        <xacro:property name="rflc"              value="-1"/>
-        <xacro:property name="base_plate"        value='base_plate_B'/>
-        <xacro:property name="servo1_holder_xyz" value=" 0.052 0.018 0.004"/>
     </xacro:if>
     <!-- ============================================================================================================================== -->
@@ -90,5 +80,5 @@
         <origin xyz="0 ${-servo_z/2-0.002} ${0.01+0.0025/2}" rpy="0 0 0"/>
         <axis xyz="0 -1 0"/>
-        <limit effort="1000.0" velocity="20.0" lower="${urdf_pi - urdf_pi/3}" upper="${urdf_pi + urdf_pi/3}"/>
+        <limit effort="1000.0" velocity="50.0" lower="${urdf_pi - urdf_pi/3}" upper="${urdf_pi + urdf_pi/3}"/>
         <dynamics friction="0.05" damping="0.1"/>
     </joint>
@@ -156,8 +146,8 @@
         <parent link="servo2_${prefix}"/>
         <child  link="servo2_padding_${prefix}"/>
-        <origin xyz="${rflc*(servo_z/2+0.002)} -0.01125 0" rpy="${-3*urdf_pi/8} 0 0"/>
-        <axis xyz="${-rflc} 0 0"/>
-        <limit effort="1000.0" velocity="20.0" lower="${urdf_pi - 2*urdf_pi/6 - rflc*urdf_pi/6}"
-                                               upper="${urdf_pi + 2*urdf_pi/6 - rflc*urdf_pi/6}"/>
+        <origin xyz="${rflc*(servo_z/2+0.002)} -0.01125 0" rpy="0 0 0"/>
+        <axis xyz="${rflc} 0 0"/>
+        <limit effort="1000.0" velocity="50.0" lower="${urdf_pi - 2*urdf_pi/6 + rflc*urdf_pi/6}"
+                                               upper="${urdf_pi + 2*urdf_pi/6 + rflc*urdf_pi/6}"/>
         <dynamics friction="0.05" damping="0.1"/>
     </joint>
@@ -169,5 +159,5 @@
             </geometry>
             <material name="blue"/>
-            <origin xyz="0 0 0" rpy="${rflc*urdf_pi/2} 0 ${-urdf_pi/2}"/>
+            <origin xyz="0 0 0" rpy="${rflc*urdf_pi/2} 0 ${urdf_pi/2}"/>
         </visual>
         <collision>
@@ -175,13 +165,13 @@
                 <box size="0.032 0.040 0.006"/>
             </geometry>
-            <origin xyz="${-rflc*0.003} -0.016 0" rpy="${rflc*urdf_pi/2} 0 ${-urdf_pi/2}"/>
+            <origin xyz="${rflc*0.003} 0.016 0" rpy="${rflc*urdf_pi/2} 0 ${urdf_pi/2}"/>
         </collision>
         <xacro:box_inertia m="0.0085" x="0.032" y="0.040" z="0.006"
-                           o_xyz="${-rflc*0.003} -0.016 0" o_rpy="${rflc*urdf_pi/2} 0 ${-urdf_pi/2}"/>
+                           o_xyz="${rflc*0.003} -0.016 0" o_rpy="${rflc*urdf_pi/2} 0 ${urdf_pi/2}"/>
     </link>
     <joint name="servo2_padding_inner_thigh_${prefix}" type="fixed">
         <parent link="servo2_padding_${prefix}"/>
         <child  link="inner_thigh_${prefix}"/>
-        <origin xyz="${rflc*0.004} 0 -0.016" rpy="${-3*urdf_pi/8} 0 ${urdf_pi}"/>
+        <origin xyz="${rflc*0.004} -0.016 0" rpy="0 0 0"/>
     </joint>
     <link name="outer_thigh_${prefix}">
@@ -191,5 +181,5 @@
             </geometry>
             <material name="blue"/>
-            <origin xyz="0 0 0" rpy="${-urdf_pi/2} ${urdf_pi/2+rflc*urdf_pi/2} ${rflc*urdf_pi/2}"/>
+            <origin xyz="0 0 0" rpy="${-urdf_pi/2} ${urdf_pi/2-rflc*urdf_pi/2} ${-rflc*urdf_pi/2}"/>
         </visual>
         <collision>
@@ -197,13 +187,13 @@
                 <box size="0.040 0.032 0.006"/>
             </geometry>
-            <origin xyz="${-rflc*0.003} -0.0475 0" rpy="${-urdf_pi/2} ${urdf_pi/2+rflc*urdf_pi/2} ${rflc*urdf_pi/2}"/>
+            <origin xyz="${rflc*0.003} -0.06 0" rpy="${-urdf_pi/2} ${urdf_pi/2-rflc*urdf_pi/2} ${-rflc*urdf_pi/2}"/>
         </collision>
         <xacro:box_inertia m="0.0113" x="0.040" y="0.032" z="0.006"
-                           o_xyz="${-rflc*0.003} -0.0475 0" o_rpy="${-urdf_pi/2} ${urdf_pi/2+rflc*urdf_pi/2} ${rflc*urdf_pi/2}"/>
+                           o_xyz="${rflc*0.003} 0.0475 0" o_rpy="${-urdf_pi/2} ${urdf_pi/2-rflc*urdf_pi/2} ${-rflc*urdf_pi/2}"/>
     </link>
     <joint name="inner_thigh_outer_thigh_${prefix}" type="fixed">
         <parent link="inner_thigh_${prefix}"/>
         <child  link="outer_thigh_${prefix}"/>
-        <origin xyz="${-rflc*0.028} 0 0" rpy="0 0 0"/>
+        <origin xyz="${rflc*0.028} 0 0" rpy="${urdf_pi} 0 0"/>
     </joint>
     <link name="servo3_${prefix}">
@@ -212,5 +202,5 @@
                 <box size="${servo_x} ${servo_y} ${servo_z}"/>
             </geometry>
-            <origin xyz="0 ${-servo_y/2} 0" rpy="0 ${-rflc*urdf_pi/2} 0"/>
+            <origin xyz="0 ${-servo_y/2} 0" rpy="0 ${rflc*urdf_pi/2} 0"/>
             <material name="black"/>
         </visual>
@@ -219,13 +209,13 @@
                 <box size="${servo_x} ${servo_y} ${servo_z}"/>
             </geometry>
-            <origin xyz="0 ${-servo_y/2} 0" rpy="0 ${-rflc*urdf_pi/2} 0"/>
+            <origin xyz="0 ${-servo_y/2} 0" rpy="0 ${rflc*urdf_pi/2} 0"/>
         </collision>
         <xacro:box_inertia m="${0.0572+0.0113+0.0078}" x="${servo_x}" y="${servo_y}" z="${servo_z}"
-                           o_xyz="0 ${-servo_y/2} 0" o_rpy="0 ${-rflc*urdf_pi/2} 0"/>
+                           o_xyz="0 ${-servo_y/2} 0" o_rpy="0 ${rflc*urdf_pi/2} 0"/>
     </link>
     <joint name="outer_thigh_servo3_${prefix}" type="fixed">
         <parent link="outer_thigh_${prefix}"/>
         <child  link="servo3_${prefix}"/>
-        <origin xyz="${-rflc*(servo_y/2-0.006-0.0025)} -0.004 0" rpy="0 0 0"/>
+        <origin xyz="${rflc*(servo_y/2-0.006-0.0025)} -0.004 0" rpy="0 0 0"/>
     </joint>
     <link name="calfFeet_${prefix}">
@@ -235,5 +225,5 @@
             </geometry>
             <material name="purple"/>
-            <origin xyz="${-0.004} -0.008 0.038" rpy="0 ${urdf_pi/2} 0"/>
+            <origin xyz="0.004 0.008 0.038" rpy="0 ${urdf_pi/2} ${urdf_pi}"/>
         </visual>
         <collision>
@@ -249,7 +239,7 @@
         <parent link="servo3_${prefix}"/>
         <child  link="calfFeet_${prefix}"/>
-        <origin xyz="${-rflc*(-servo_z/2-0.002-0.0025)} ${-0.086+0.004} 0" rpy="0 0 0"/>
+        <origin xyz="${rflc*(-servo_z/2-0.002-0.0025)} ${-0.086+0.004} 0" rpy="${urdf_pi} 0 0"/>
         <axis xyz="${-rflc} 0 0"/>
-        <limit effort="1000.0" velocity="20.0" lower="${5*urdf_pi/8}" upper="${11*urdf_pi/8}"/>
+        <limit effort="1000.0" velocity="50.0" lower="${5*urdf_pi/8}" upper="${11*urdf_pi/8}"/>
         <dynamics friction="0.0128" damping="0.1"/>
     </joint>
@@ -259,5 +249,5 @@
                 <mesh filename="package://my_robot_description/mesh/CADv1/calfJoint.stl" scale="0.001 0.001 0.001"/>
             </geometry>
-            <origin xyz="0 0 0" rpy="${urdf_pi/2} 0 ${rflc*urdf_pi/2}"/>
+            <origin xyz="0 0 0" rpy="${-urdf_pi/2} 0 ${rflc*urdf_pi/2}"/>
             <material name="white"/>
         </visual>
@@ -266,16 +256,16 @@
                 <box size="0.022 0.053 0.007"/>
             </geometry>
-            <origin xyz="${rflc*0.0005} 0 0.0155" rpy="${urdf_pi/2} 0 ${rflc*urdf_pi/2}"/>
+            <origin xyz="${-rflc*0.0005} 0 -0.0155" rpy="${-urdf_pi/2} 0 ${-rflc*urdf_pi/2}"/>
         </collision>
         <xacro:box_inertia m="${0.0047+0.0015}" x="0.022" y="0.053" z="0.007"
-                           o_xyz="${rflc*0.0005} 0 0.0155" o_rpy="${urdf_pi/2} 0 ${rflc*urdf_pi/2}"/>
+                           o_xyz="${-rflc*0.0005} 0 -0.0155" o_rpy="${-urdf_pi/2} 0 ${-rflc*urdf_pi/2}"/>
     </link>
     <joint name="servo3_calfJoint_${prefix}" type="revolute">
         <parent link="servo3_${prefix}"/>
         <child  link="calfJoint_${prefix}"/>
-        <origin xyz="${-rflc*(-servo_z/2-0.002-0.0025)} ${-0.01-0.0025/2} 0" rpy="0 0 0"/>
+        <origin xyz="${rflc*(-servo_z/2-0.002-0.0025)} ${-0.01-0.0025/2} 0" rpy="0 0 0"/>
         <axis xyz="${-rflc} 0 0"/>
         <mimic joint="servo3_calfFeet_${prefix}" multiplier="1.0" offset="0.0"/>
-        <limit effort="1000.0" velocity="20.0" lower="${5*urdf_pi/8}" upper="${11*urdf_pi/8}"/>
+        <limit effort="1000.0" velocity="50.0" lower="${5*urdf_pi/8}" upper="${11*urdf_pi/8}"/>
         <dynamics friction="0.0212" damping="0.1"/>
     </joint>
@@ -299,5 +289,5 @@
         <parent link="calfFeet_${prefix}"/>
         <child  link="calfSphere_${prefix}"/>
-        <origin xyz="0 0.004 ${-0.105+0.035}" rpy="0 0 0"/>
+        <origin xyz="0 -0.004 ${-0.105+0.035}" rpy="0 0 0"/>
     </joint>
     </xacro:macro>

File: src/my_robot_description/urdf/cubic_doggo_legF.xacro (robot description, xacro)
@@ -16,14 +16,4 @@
         <xacro:property name="servo1_holder_xyz" value=" 0.052 0.018 0.004"/>
     </xacro:if>
-    <xacro:if value="${prefix == 'BL'}">
-        <xacro:property name="rflc"              value=" 1"/>
-        <xacro:property name="base_plate"        value='base_plate_B'/>
-        <xacro:property name="servo1_holder_xyz" value="-0.052 0.018 0.004"/>
-    </xacro:if>
-    <xacro:if value="${prefix == 'BR'}">
-        <xacro:property name="rflc"              value="-1"/>
-        <xacro:property name="base_plate"        value='base_plate_B'/>
-        <xacro:property name="servo1_holder_xyz" value=" 0.052 0.018 0.004"/>
-    </xacro:if>
     <!-- ============================================================================================================================== -->
     <link name="servo1_holder_${prefix}">
@@ -90,5 +80,5 @@
         <origin xyz="0 ${-servo_z/2-0.002} ${0.01+0.0025/2}" rpy="0 0 0"/>
         <axis xyz="0 -1 0"/>
-        <limit effort="1000.0" velocity="20.0" lower="${urdf_pi - urdf_pi/3}" upper="${urdf_pi + urdf_pi/3}"/>
+        <limit effort="1000.0" velocity="50.0" lower="${urdf_pi - urdf_pi/3}" upper="${urdf_pi + urdf_pi/3}"/>
         <dynamics friction="0.05" damping="0.1"/>
     </joint>
@@ -129,5 +119,6 @@
             <origin xyz="0 ${-servo_y/2} 0" rpy="0 ${rflc*urdf_pi/2} 0"/>
         </collision>
-        <xacro:box_inertia m="0.0572" x="${servo_x}" y="${servo_y}" z="${servo_z}" o_xyz="0 ${-servo_y/2} 0" o_rpy="0 ${rflc*urdf_pi/2} 0"/>
+        <xacro:box_inertia m="0.0572" x="${servo_x}" y="${servo_y}" z="${servo_z}"
+                           o_xyz="0 ${-servo_y/2} 0" o_rpy="0 ${rflc*urdf_pi/2} 0"/>
     </link>
     <joint name="servo2_holder_servo2_${prefix}" type="fixed">
@@ -157,5 +148,5 @@
         <origin xyz="${rflc*(servo_z/2+0.002)} -0.03525 0" rpy="0 0 0"/>
         <axis xyz="${rflc} 0 0"/>
-        <limit effort="1000.0" velocity="20.0" lower="${urdf_pi - 2*urdf_pi/6 - rflc*urdf_pi/6}"
+        <limit effort="1000.0" velocity="50.0" lower="${urdf_pi - 2*urdf_pi/6 - rflc*urdf_pi/6}"
                                                upper="${urdf_pi + 2*urdf_pi/6 - rflc*urdf_pi/6}"/>
         <dynamics friction="0.05" damping="0.1"/>
@@ -196,5 +187,5 @@
                 <box size="0.040 0.032 0.006"/>
             </geometry>
-            <origin xyz="${rflc*0.003} -0.0475 0" rpy="${-urdf_pi/2} ${urdf_pi/2-rflc*urdf_pi/2} ${-rflc*urdf_pi/2}"/>
+            <origin xyz="${rflc*0.003} -0.06 0" rpy="${-urdf_pi/2} ${urdf_pi/2-rflc*urdf_pi/2} ${-rflc*urdf_pi/2}"/>
         </collision>
         <xacro:box_inertia m="0.0113" x="0.040" y="0.032" z="0.006"
@@ -250,5 +241,5 @@
         <origin xyz="${rflc*(-servo_z/2-0.002-0.0025)} ${-0.086+0.004} 0" rpy="0 0 0"/>
         <axis xyz="${-rflc} 0 0"/>
-        <limit effort="1000.0" velocity="20.0" lower="${5*urdf_pi/8}" upper="${11*urdf_pi/8}"/>
+        <limit effort="1000.0" velocity="50.0" lower="${5*urdf_pi/8}" upper="${11*urdf_pi/8}"/>
         <dynamics friction="0.0128" damping="0.1"/>
     </joint>
@@ -273,8 +264,8 @@
         <parent link="servo3_${prefix}"/>
         <child  link="calfJoint_${prefix}"/>
-        <origin xyz="${rflc*(-servo_z/2-0.002-0.0025)} ${-0.01-0.0025/2} 0" rpy="0 0 0"/>
+        <origin xyz="${rflc*(-servo_z/2-0.002-0.0025)} ${-0.01-0.0025/2-0.001} 0" rpy="0 0 0"/>
         <axis xyz="${-rflc} 0 0"/>
         <mimic joint="servo3_calfFeet_${prefix}" multiplier="1.0" offset="0.0"/>
-        <limit effort="1000.0" velocity="20.0" lower="${5*urdf_pi/8}" upper="${11*urdf_pi/8}"/>
+        <limit effort="1000.0" velocity="50.0" lower="${5*urdf_pi/8}" upper="${11*urdf_pi/8}"/>
         <dynamics friction="0.0212" damping="0.1"/>
     </joint>
